File: RheoBoard_PCB/RheoBoard_v1.05/RheoboardV1/1.kicad_pcb (KiCad board)
At the start: 2 copper layers, 109 x 126.4 mm, 160 parts, among them J1 JST SH 4-pin 1.00mm, J12 JST SH 4-pin 1.00mm, J17 JST SH 4-pin 1.00mm, J18 JST EH 3-pin 2.50mm, J2 PJ-082BH, J3 JST EH 4-pin 2.50mm, J9 JST SH 4-pin 1.00mm, Q10 AO3400A, Q3 AO3400A, Q4 AO3400A, Q8 AO3400A, SW1 TL3301NF160QG/P010515, SW2 TL3301NF160QG/P010515, SW3 TL3301NF160QG/P010515, SW4 TL3301NF160QG/P010515, U1 TPS563203DRLR, U10 JST XH 2-pin 2.50mm, U11 ZR370-02PM / 4.5V / 2.5 LPM /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, U12 TPS259472ARPWR, U2 TPS563203DRLR, U3 TPS563203DRLR, U4 TCA9534APWR, U5 MPRLS0025PA00001A, U7 PCA9685PW,118, U8 ZR370-02PM / 4.5V / 2.5 LPM /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, U9 JST XH 2-pin 2.50mm

Commit message: Update documentation for RheoBoard version 2
- Revised `CHANGELOG.md`, `README.md`, and `BuildYourOwn/README.md` to clarify the transition to a 3D-printed panel, removing references to the previous laser-cut design.
- Updated `okh-RheoBoard.yml` to reflect the current version and its status, ensuring consistency across documentation.
- Enhanced clarity regarding the assembly instructions and parts list, emphasizing the new design and providing updated links to relevant files.

These updates improve user understanding of the project's evolution and provide comprehensive guidance for building and using the RheoBoard.
Parts:
- added C68: 100nF 50V X7R ±10%, Capacitor_SMD:C_0603_1608Metric_Pad1.08x0.95mm_HandSolder, F.Cu at (189.0, 109.0)
- added C69: 100nF 50V X7R ±10%, Capacitor_SMD:C_0603_1608Metric_Pad1.08x0.95mm_HandSolder, F.Cu at (193.0, 109.0)
- added R82: 4K7/0603/1%, Resistor_SMD:R_0603_1608Metric_Pad0.98x0.95mm_HandSolder, F.Cu at (190.0, 117.0)
- added R83: 4K7/0603/1%, Resistor_SMD:R_0603_1608Metric_Pad0.98x0.95mm_HandSolder, F.Cu at (192.5, 117.0)
- added R84: 10K/0603/1%, Resistor_SMD:R_0603_1608Metric_Pad0.98x0.95mm_HandSolder, F.Cu at (195.5, 114.0)
- added U13: TCA9517ADGKR, RheoBoard:TI_DGK0008A_VSSOP_3x3mm_P0.65mm, F.Cu at (190.8, 112.0)
Connections:
- J9 pad 2: +3V3 -> /HOST_3V3
- J9 pad 3: /SDA -> /HOST_SDA
- J9 pad 4: /SCL -> /HOST_SCL
Routing:
- net /HOST_3V3: track 0.00 -> 37.0 mm, vias 0 -> 2
- net /HOST_SCL: track 0.00 -> 16.2 mm, vias 0 -> 4
- net /HOST_SDA: track 0.00 -> 15.3 mm
- net /SDA: track 278.7 -> 291.2 mm, vias 8 -> 9
- net /SCL: track 290.1 -> 294.6 mm, vias 7 -> 8
- net GND: track 12.3 -> 16.6 mm, vias 220 -> 218
- net +3V3: track 337.2 -> 334.9 mm, vias 13 -> 11
Other:
- board text added: "C69"
- board text added: "HOST 3V3 IN"
- board text added: "LOCAL SERVICE"
- board text added: "QWIIC MASTER"
- board text added: "QWIIC SENSOR"
- board text added: "R83"
- board text added: "R84"
- board text added: "U13"
- board text removed: "I2C_1"
- board text removed: "I2C_2"
- board text removed: "I2C_3"
- board text removed: "I2C_4"
- board text removed: "MASTER / MUX"

Commit message: Remove redundant J18 header and update documentation for RheoBoard v1.05
- Removed the J18 local service header from the PCB design, as it is no longer needed.
- Updated the assembly instructions to reflect the removal of J18 and clarified the role of J3 as the local debug header.
- Revised the README and BOM to indicate the changes in the connector layout and part count.
- Adjusted the Gerber files and other manufacturing documents to ensure consistency with the updated design.

These changes streamline the design and improve the clarity of the documentation for users and manufacturers.
Parts:
- removed J18: JST EH 3-pin 2.50mm, Connector_JST:JST_EH_B3B-EH-A_1x03_P2.50mm_Vertical
Routing:
- net /SCL: track 294.6 -> 233.6 mm
- net /SDA: track 291.2 -> 235.8 mm
Other:
- board text removed: "GND SDA SCL"
- board text removed: "J18"
- board text removed: "LOCAL SERVICE"
