File: RheoBoard_PCB/RheoBoard_v1.05/RheoboardV1/1.kicad_sch (KiCad schematic)
At the start: 160 parts, among them J1 JST SH 4-pin 1.00mm, J12 JST SH 4-pin 1.00mm, J17 JST SH 4-pin 1.00mm, J18 JST EH 3-pin 2.50mm, J2 PJ-082BH, J3 JST EH 4-pin 2.50mm, J9 JST SH 4-pin 1.00mm, Q10 AO3400A, Q3 AO3400A, Q4 AO3400A, Q8 AO3400A, SW1 TL3301NF160QG/P010515, SW2 TL3301NF160QG/P010515, SW3 TL3301NF160QG/P010515, SW4 TL3301NF160QG/P010515, U1 TPS563203DRLR, U10 JST XH 2-pin 2.50mm, U11 ZR370-02PM / 4.5V / 2.5 LPM /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, U12 TPS259472ARPWR, U2 TPS563203DRLR, U3 TPS563203DRLR, U4 TCA9534APWR, U5 MPRLS0025PA00001A, U7 PCA9685PW,118, U8 ZR370-02PM / 4.5V / 2.5 LPM /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, U9 JST XH 2-pin 2.50mm

Commit message: Update documentation for RheoBoard version 2
- Revised `CHANGELOG.md`, `README.md`, and `BuildYourOwn/README.md` to clarify the transition to a 3D-printed panel, removing references to the previous laser-cut design.
- Updated `okh-RheoBoard.yml` to reflect the current version and its status, ensuring consistency across documentation.
- Enhanced clarity regarding the assembly instructions and parts list, emphasizing the new design and providing updated links to relevant files.

These updates improve user understanding of the project's evolution and provide comprehensive guidance for building and using the RheoBoard.
Parts:
- added C68, C69: 100nF 50V X7R ±10%, Capacitor_SMD:C_0603_1608Metric_Pad1.08x0.95mm_HandSolder, symbol Device:C
- added R82, R83: 4K7/0603/1%, Resistor_SMD:R_0603_1608Metric_Pad0.98x0.95mm_HandSolder, symbol Device:R_US
- added R84: 10K/0603/1%, Resistor_SMD:R_0603_1608Metric_Pad0.98x0.95mm_HandSolder, symbol Device:R_US
- added U13: TCA9517ADGKR, RheoBoard:TI_DGK0008A_VSSOP_3x3mm_P0.65mm, symbol Logic_LevelTranslator:TCA9517ADGK
- J1, J12, J17: Role (none) -> QWIIC SENSOR: local RheoBoard +3V3 power output
- J18: Role (none) -> LOCAL BUS SERVICE: GND/SDA/SCL; no supply pin
- J9: Role (none) -> QWIIC MASTER: independently powered ESP32 Thing Plus; pin2 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
Connections:
- net +3V3: now also C68.1, U13.1 (VCCA); no longer J9.2 (Pin_2)
- net GND: now also C68.2, C69.2, R84.2, U13.4 (GND)
- net SCL: now also U13.2 (SCLA); no longer J9.4 (Pin_4)
- net SDA: now also U13.3 (SDAA); no longer J9.3 (Pin_3)
- new net HOST_3V3: C69.1, J9.2 (Pin_2), R82.1, R83.1, R84.1, U13.5 (EN), U13.8 (VCCB)
- new net HOST_SCL: J9.4 (Pin_4), R83.2, U13.7 (SCLB)
- new net HOST_SDA: J9.3 (Pin_3), R82.2, U13.6 (SDAB)
Other:
- note added: "J18: LOCAL SERVICE BUS (GND / SDA / SCL); no power-domain isolation. J9: dedicated standard Qwiic master port. J1 / J12 / J17: powered sensors. Multiple boards: external TCA9548A at 0x71; one channel active. Disable PCA9685 ALLCALL after initialization."
- note added: "LOCAL A: RheoBoard +3V3 and sensor bus HOST B: ESP32-supplied +3V3; regulators never paralleled 100 kHz initial bring-up; cable/module pull-ups share a current budget J1 / J12 / J17 remain powered Qwiic sensor ports J18 = LOCAL BUS SERVICE; no master-power isolation at that header"
- note added: "QWIIC MASTER: J9 TO USB / BATTERY ESP32"
- note removed: "MASTER / EXTERNAL MUX: GND, SDA, SCL only Each board powered from its own 12 V input. Existing 4-pin ports: local 3V3 OUTPUT for peripherals. Multiple boards: TCA9548A at 0x71, one channel active. Disable PCA9685 ALLCALL after initialization."

Commit message: Remove redundant J18 header and update documentation for RheoBoard v1.05
- Removed the J18 local service header from the PCB design, as it is no longer needed.
- Updated the assembly instructions to reflect the removal of J18 and clarified the role of J3 as the local debug header.
- Revised the README and BOM to indicate the changes in the connector layout and part count.
- Adjusted the Gerber files and other manufacturing documents to ensure consistency with the updated design.

These changes streamline the design and improve the clarity of the documentation for users and manufacturers.
Parts:
- removed J18: JST EH 3-pin 2.50mm, Connector_JST:JST_EH_B3B-EH-A_1x03_P2.50mm_Vertical, symbol Connector_Generic:Conn_01x03
Other:
- note added: "J3: LOCAL DEBUG BUS (GND / +3V3 / SDA / SCL); onboard supply. J9: dedicated standard Qwiic master port. J1 / J12 / J17: powered sensors. Multiple boards: external TCA9548A at 0x71; one channel active. Disable PCA9685 ALLCALL after initialization."
- note added: "LOCAL A: RheoBoard +3V3 and sensor bus HOST B: ESP32-supplied +3V3; regulators never paralleled 100 kHz initial bring-up; cable/module pull-ups share a current budget J1 / J12 / J17 remain powered Qwiic sensor ports J3 = LOCAL DEBUG BUS; no master-power isolation at that header"
- note removed: "J18: LOCAL SERVICE BUS (GND / SDA / SCL); no power-domain isolation. J9: dedicated standard Qwiic master port. J1 / J12 / J17: powered sensors. Multiple boards: external TCA9548A at 0x71; one channel active. Disable PCA9685 ALLCALL after initialization."
- note removed: "LOCAL A: RheoBoard +3V3 and sensor bus HOST B: ESP32-supplied +3V3; regulators never paralleled 100 kHz initial bring-up; cable/module pull-ups share a current budget J1 / J12 / J17 remain powered Qwiic sensor ports J18 = LOCAL BUS SERVICE; no master-power isolation at that header"
Changed lines of the file:
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@@
 	(wire
 		(pts
-			(xy 756.92 210.82)
-			(xy 754.38 210.82)
-		)
-	)
-	(wire
-		(pts
-			(xy 756.92 213.36)
-			(xy 754.38 213.36)
-		)
-	)
-	(wire
-		(pts
-			(xy 756.92 215.9)
-			(xy 754.38 215.9)
-		)
-	)
-	(wire
-		(pts
-			(xy 754.38 210.82)
-			(xy 754.38 207.01)
-		)
-	)
-	(wire
-		(pts
 			(xy 529.59 426.72)
 			(xy 529.59 434.34)
@@
 		)
 	)
-	(text "LOCAL A: RheoBoard +3V3 and sensor bus\nHOST B: ESP32-supplied +3V3; regulators never paralleled\n100 kHz initial bring-up; cable/module pull-ups share a current budget\nJ1 / J12 / J17 remain powered Qwiic sensor ports\nJ18 = LOCAL BUS SERVICE; no master-power isolation at that header"
-		(at 643.89 340.36 0)
-		(effects
-			(font
-				(size 1.27 1.27)
-			)
-			(justify left bottom)
-		)
-	)
 	(text "QWIIC MASTER: J9 TO USB / BATTERY ESP32"
 		(at 643.89 285.75 0)
@@
 		)
 	)
-	(text "J18: LOCAL SERVICE BUS (GND / SDA / SCL); no power-domain isolation.\nJ9: dedicated standard Qwiic master port. J1 / J12 / J17: powered sensors.\nMultiple boards: external TCA9548A at 0x71; one channel active.\nDisable PCA9685 ALLCALL after initialization."
-		(at 640.08 254 0)
-		(effects
-			(font
-				(size 1.27 1.27)
-			)
-			(justify left bottom)
-		)
-	)
-	(label "SDA"
-		(at 754.38 213.36 180)
-		(effects
-			(font
-				(size 1.27 1.27)
-			)
-			(justify right bottom)
-		)
-	)
-	(label "SCL"
-		(at 754.38 215.9 180)
-		(effects
-			(font
-				(size 1.27 1.27)
-			)
-			(justify right bottom)
-		)
-	)
 	(label "EF_EN"
 		(at 358.14 162.56 180)
@@
 		)
 	)
-	(global_label "GND"
-		(shape input)
-		(at 754.38 207.01 0)
-		(effects
-			(font
-				(size 1.27 1.27)
-			)
-			(justify left)
-		)
-	)
 	(global_label "PUMP1_PWM"
 		(shape input)
@@
 		)
 	)
+  (text "J3: LOCAL DEBUG BUS (GND / +3V3 / SDA / SCL); onboard supply.\nJ9: dedicated standard Qwiic master port. J1 / J12 / J17: powered sensors.\nMultiple boards: external TCA9548A at 0x71; one channel active.\nDisable PCA9685 ALLCALL after initialization."
+    (at 640.08 254 0)
+    (effects (font (size 1.27 1.27)) (justify left bottom))
+  )
+  (text "LOCAL A: RheoBoard +3V3 and sensor bus\nHOST B: ESP32-supplied +3V3; regulators never paralleled\n100 kHz initial bring-up; cable/module pull-ups share a current budget\nJ1 / J12 / J17 remain powered Qwiic sensor ports\nJ3 = LOCAL DEBUG BUS; no master-power isolation at that header"
+    (at 643.89 340.36 0)
+    (effects (font (size 1.27 1.27)) (justify left bottom))
+  )
 	(symbol
 		(lib_id "Mechanical:MountingHole")
@@
 					(unit 1)
 				)
-			)
-		)
-	)
-	(symbol
-		(lib_id "Connector_Generic:Conn_01x03")
-		(at 762 213.36 0)
-		(unit 1)
-		(in_bom yes)
-		(on_board yes)
-		(dnp no)
-		(property "Reference" "J18"
-			(at 769.62 209.55 0)
-			(effects
-				(font
-					(size 1.27 1.27)
-				)
-			)
-		)
-		(property "Value" "JST EH 3-pin 2.50mm"
-			(at 762 218.44 0)
-			(effects
-				(font
-					(size 1.27 1.27)
-				)
-			)
-		)
-		(property "Footprint" "Connector_JST:JST_EH_B3B-EH-A_1x03_P2.50mm_Vertical"
-			(at 762 213.36 0)
-			(hide yes)
-			(effects
-				(font
-					(size 1.27 1.27)
-				)
-			)
-		)
-		(property "Datasheet" "https://www.jst-mfg.com/product/pdf/eng/eEH.pdf"
-			(at 762 213.36 0)
-			(hide yes)
-			(effects
-				(font
-					(size 1.27 1.27)
-				)
-			)
-		)
-		(property "Description" "Generic connector, single row, 01x03, script generated (kicad-library-utils/schlib/autogen/connector/)"
-			(at 762 213.36 0)
-			(hide yes)
-			(effects
-				(font
-					(size 1.27 1.27)
-				)
-			)
-		)
-		(property "Assembly" "Manual THT"
-			(at 762 213.36 0)
-			(hide yes)
-			(effects
-				(font
-					(size 1.27 1.27)
-				)
-			)
-		)
-		(property "LCSC" "C160259"
-			(at 762 213.36 0)
-			(hide yes)
-			(effects
-				(font
-					(size 1.27 1.27)
-				)
-			)
-		)
-		(property "MPN" "B3B-EH-A(LF)(SN)"
-			(at 762 213.36 0)
-			(hide yes)
-			(effects
-				(font
-					(size 1.27 1.27)
-				)
-			)
-		)
-		(property "Manufacturer" "JST"
-			(at 762 213.36 0)
-			(hide yes)
-			(effects
-				(font
-					(size 1.27 1.27)
-				)
-			)
-		)
-		(property "Source" "https://www.lcsc.com/product-detail/C160259.html"
-			(at 762 213.36 0)
-			(hide yes)
-			(effects
-				(font
-					(size 1.27 1.27)
-				)
-			)
-		)
-		(property "Role" "LOCAL BUS SERVICE: GND/SDA/SCL; no supply pin"
-			(at 762 213.36 0)
-			(hide yes)
-			(effects
-				(font
-					(size 1.27 1.27)
-				)
-			)
-		)
-		(instances
-			(project "1"
-				(path "/5b05ede3-198a-4bf9-b0d8-5fef5c8d1378"
-					(reference "J18")
-					(unit 1)
-				)
