File: RheoBoard_PCB/RheoBoard_v1.05/RheoboardV1/RheoBoard_v1.05.kicad_sch (KiCad schematic)
At the start: 167 parts, among them J1 JST SH 4-pin 1.00mm, J12 JST SH 4-pin 1.00mm, J17 JST SH 4-pin 1.00mm, J2 PJ-082BH, J3 JST EH 4-pin 2.50mm, J9 JST SH 4-pin 1.00mm, Q10 AO3400A, Q11 DMP6023LE-13, Q3 AO3400A, Q4 AO3400A, Q8 AO3400A, SW1 TL3301NF160QG/P010515, SW2 TL3301NF160QG/P010515, SW3 TL3301NF160QG/P010515, SW4 TL3301NF160QG/P010515, U1 TPS563203DRLR, U10 JST XH 2-pin 2.50mm, U11 ZR370-02PM / 4.5V / 2.5 LPM /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, U12 TPS259472ARPWR, U13 TCA9517ADGKR, U2 TPS563203DRLR, U3 TPS563203DRLR, U4 TCA9534APWR, U5 MPRLS0025PA00001A, U7 PCA9685PW,118, U8 ZR370-02PM / 4.5V / 2.5 LPM /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, U9 JST XH 2-pin 2.50mm

Commit message: Update documentation and references for RheoBoardOTS and RheoBoard_v1
- Revised README files to consistently refer to RheoBoardOTS - DIY and RheoBoard_v1 - PCB, enhancing clarity for users.
- Updated assembly and wiring documentation to reflect the new naming conventions and ensure accurate references across all sections.
- Adjusted safety and firmware documentation to specify the application of RheoData for the updated project versions.
- Enhanced image references and descriptions to align with the latest design changes.

These updates improve the organization, usability, and clarity of the RheoBoard project documentation.
Parts:
- removed C22: 10nF 50V ±10%, Capacitor_SMD:C_0603_1608Metric_Pad1.08x0.95mm_HandSolder, symbol Device:C
- removed C47: 100nF 50V X7R ±10%, Capacitor_SMD:C_0603_1608Metric_Pad1.08x0.95mm_HandSolder, symbol Device:C
- removed R10: 2K2/0603/1%, Resistor_SMD:R_0603_1608Metric_Pad0.98x0.95mm_HandSolder, symbol Device:R_US
- removed R11: 4K7/0603/1%, Resistor_SMD:R_0603_1608Metric_Pad0.98x0.95mm_HandSolder, symbol Device:R_US
- removed R13, R14: 10K/0603/1%, Resistor_SMD:R_0603_1608Metric_Pad0.98x0.95mm_HandSolder, symbol Device:R_US
- removed TP1: TestPoint, TestPoint:TestPoint_Pad_D1.0mm, symbol Connector:TestPoint_Alt
- removed U4: TCA9534APWR, RheoBoard:TCA9534APWR, symbol Rheo_TCA9534APWR:TCA9534APWR
- added J19: BUTTONS_GPIO, Connector_PinHeader_2.54mm:PinHeader_1x05_P2.54mm_Vertical, symbol Connector_Generic:Conn_01x05
Connections:
- net +3V3: no longer R16.1, R17.1, R18.1, R19.1
- net HOST_3V3: now also R16.1, R17.1, R18.1, R19.1
- net VALVE1: now also U7.11 (PWM5)
- net VALVE2: now also U7.12 (PWM6)
- no-connect marks 15 -> 13

Commit message: Update documentation and design files for RheoBoard project
- Revised README.md to enhance clarity on build instructions and component descriptions for RheoBoardOTS - DIY and RheoBoard_v1 - PCB.
- Updated hardware documentation to include detailed specifications for the Cysljoyful AC/DC adapter and its role in the system.
- Enhanced image references and descriptions to align with the latest design changes, including the addition of new images for the power adapter.
- Adjusted schematic and PCB files to improve component alignment and clarity, including the addition of new wire connections and labels.

These updates improve the organization, usability, and clarity of the RheoBoard project documentation and design files.
Connections:
- net GND: now also J19.1 (Pin_1)
- net PUMP1_IN: now also J19.4 (Pin_4)
- net PUMP2_IN: now also J19.5 (Pin_5)
- net VALVE1_IN: now also J19.2 (Pin_2)
- net VALVE2_IN: now also J19.3 (Pin_3)
Other:
- note added: "BUTTON GPIO TO ESP32"
- note added: "J19 pin 1: GND; pins 2-5: SW1, SW2, SW3, SW4. Active-low; connect J9 Qwiic cable for HOST_3V3 pull-ups. Suggested ESP32 GPIOs: 32, 33, 25, 26 respectively."
- note added: "Valve channels 5/6: full ON / full OFF only."
Changed lines of the file:
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@@
 		)
 	)
+	(wire
+		(pts
+			(xy 495.3 88.9)
+			(xy 505.46 88.9)
+		)
+	)
+	(wire
+		(pts
+			(xy 495.3 91.44)
+			(xy 505.46 91.44)
+		)
+	)
+	(wire
+		(pts
+			(xy 495.3 93.98)
+			(xy 505.46 93.98)
+		)
+	)
+	(wire
+		(pts
+			(xy 495.3 96.52)
+			(xy 505.46 96.52)
+		)
+	)
+	(wire
+		(pts
+			(xy 495.3 99.06)
+			(xy 505.46 99.06)
+		)
+	)
 	(text "BUCK 12V - 3V3\n\n"
 		(at 168.656 206.502 0)
@@
 		)
 	)
+	(text "BUTTON GPIO TO ESP32"
+		(at 478.79 76.2 0)
+		(effects
+			(font
+				(size 1.27 1.27)
+			)
+			(justify left bottom)
+		)
+	)
+	(text "J19 pin 1: GND; pins 2-5: SW1, SW2, SW3, SW4.\nActive-low; connect J9 Qwiic cable for HOST_3V3 pull-ups.\nSuggested ESP32 GPIOs: 32, 33, 25, 26 respectively."
+		(at 478.79 118.11 0)
+		(effects
+			(font
+				(size 1.27 1.27)
+			)
+			(justify left bottom)
+		)
+	)
 	(label "EF_EN"
 		(at 358.14 162.56 180)
@@
 		)
 	)
+	(label "HOST_3V3"
+		(at 485.14 393.7 90)
+		(effects
+			(font
+				(size 1.27 1.27)
+			)
+			(justify left bottom)
+		)
+	)
+	(label "HOST_3V3"
+		(at 529.59 393.7 90)
+		(effects
+			(font
+				(size 1.27 1.27)
+			)
+			(justify left bottom)
+		)
+	)
+	(label "HOST_3V3"
+		(at 574.04 393.7 90)
+		(effects
+			(font
+				(size 1.27 1.27)
+			)
+			(justify left bottom)
+		)
+	)
+	(label "HOST_3V3"
+		(at 619.76 393.7 90)
+		(effects
+			(font
+				(size 1.27 1.27)
+			)
+			(justify left bottom)
+		)
+	)
 	(global_label "VALVE2_IN"
 		(shape input)
@@
 		)
 	)
-	(global_label "HOST_3V3"
-		(shape input)
-		(at 485.14 393.7 90)
+	(global_label "VALVE1"
+		(shape output)
+		(at 722.63 96.52 0)
 		(effects
 			(font
@@
 		)
 	)
-	(global_label "HOST_3V3"
-		(shape input)
-		(at 529.59 393.7 90)
+	(global_label "VALVE2"
+		(shape output)
+		(at 722.63 99.06 0)
 		(effects
 			(font
@@
 		)
 	)
-	(global_label "HOST_3V3"
+	(global_label "GND"
 		(shape input)
-		(at 574.04 393.7 90)
+		(at 495.3 88.9 180)
 		(effects
 			(font
 				(size 1.27 1.27)
 			)
-			(justify left)
+			(justify right)
 		)
 	)
-	(global_label "HOST_3V3"
+	(global_label "VALVE1_IN"
 		(shape input)
-		(at 619.76 393.7 90)
+		(at 495.3 91.44 180)
 		(effects
 			(font
 				(size 1.27 1.27)
 			)
-			(justify left)
+			(justify right)
 		)
 	)
-	(global_label "VALVE1"
-		(shape output)
-		(at 722.63 96.52 0)
+	(global_label "VALVE2_IN"
+		(shape input)
+		(at 495.3 93.98 180)
 		(effects
 			(font
 				(size 1.27 1.27)
 			)
-			(justify left)
+			(justify right)
 		)
 	)
-	(global_label "VALVE2"
-		(shape output)
-		(at 722.63 99.06 0)
+	(global_label "PUMP1_IN"
+		(shape input)
+		(at 495.3 96.52 180)
 		(effects
 			(font
 				(size 1.27 1.27)
 			)
-			(justify left)
+			(justify right)
 		)
 	)
+	(global_label "PUMP2_IN"
+		(shape input)
+		(at 495.3 99.06 180)
+		(effects
+			(font
+				(size 1.27 1.27)
+			)
+			(justify right)
+		)
+	)
+  (text "Valve channels 5/6: full ON / full OFF only."
+    (at 669.29 133.35 0)
+    (effects (font (size 1.27 1.27)) (justify left bottom))
+  )
 	(symbol
 		(lib_id "Mechanical:MountingHole")
@@
 			)
 		)
-		(instances
-			(project "RheoBoard_v1.05"
-				(path "/5b05ede3-198a-4bf9-b0d8-5fef5c8d1378"
-					(reference "J19")
-					(unit 1)
-				)
-			)
-		)
 		(property "Assembly" "Manual"
 			(at 510.54 93.98 0)
@@
 				)
 			)
-		))
+		)
+		(instances
+			(project "RheoBoard_v1.05"
+				(path "/5b05ede3-198a-4bf9-b0d8-5fef5c8d1378"
+					(reference "J19")
+					(unit 1)
+				)
+			)
+		)
+	)
 	(rectangle
 		(start 175.26 314.706)
