File: RheoBoard_PCB/RheoBoard_v1/RheoboardV1/RheoBoard_v1.kicad_pcb (KiCad board)
At the start: 2 copper layers, 109 x 126.4 mm, 149 parts, among them J1 I2C_4, J12 I2C_2, J17 I2C_3, J2 PJ-082BH, J3 I2C_5, J9 I2C_1, Q10 AO3400A, Q3 AO3400A, Q4 AO3400A, Q8 AO3400A, SW1 SW2, SW2 SW2, SW3 SW2, SW4 SW2, U1 TPS563203DRLR, U10 VALVE2, U11 PUMP, U2 TPS563203DRLR, U3 TPS563203DRLR, U4 TCA9534APWR, U5 MPRLS0025PA00001A, U7 PCA9685, U8 PUMP, U9 VALVE

Commit message: Refactor RheoBoard v1.05 schematic and layout files. Removed redundant via definitions to streamline the PCB design. Updated schematic presentation for improved clarity and alignment, including adjustments to component placements and designators. Enhanced revision notes to reflect recent layout changes and component updates.
Routing:
- net GND: vias 210 -> 205
