File: RheoBoard_PCB/RheoBoard_v1.05/RheoBoard_v1.05/RheoBoard_v1.05.kicad_sch (KiCad schematic)
At the start: 160 parts, among them J1 JST SH 4-pin 1.00mm, J12 JST SH 4-pin 1.00mm, J17 JST SH 4-pin 1.00mm, J19 BUTTONS_GPIO, J2 PJ-082BH, J3 JST EH 4-pin 2.50mm, J9 JST SH 4-pin 1.00mm, Q10 AO3400A, Q11 DMP6023LE-13, Q3 AO3400A, Q4 AO3400A, Q8 AO3400A, SW1 TL3301NF160QG/P010515, SW2 TL3301NF160QG/P010515, SW3 TL3301NF160QG/P010515, SW4 TL3301NF160QG/P010515, U1 TPS563203DRLR, U10 JST XH 2-pin 2.50mm, U11 ZR370-02PM / 4.5V / 2.5 LPM /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, U12 TPS259472ARPWR, U13 TCA9517ADGKR, U2 TPS563203DRLR, U3 TPS563203DRLR, U5 MPRLS0025PA00001A, U7 PCA9685PW,118, U8 ZR370-02PM / 4.5V / 2.5 LPM /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, U9 JST XH 2-pin 2.50mm

Commit message: Refactor RheoBoard v1.05 schematic and layout files. Removed redundant via definitions to streamline the PCB design. Updated schematic presentation for improved clarity and alignment, including adjustments to component placements and designators. Enhanced revision notes to reflect recent layout changes and component updates.
Other:
- note added: "Input Protection"
- note added: "J9 TO USB / BATTERY ESP32"
- note added: "Qwiic Master Interface"
- note removed: "QWIIC MASTER: J9 TO USB / BATTERY ESP32"
- moved on the sheet: C23, C24, C25, C26, C27, C28, C29, C30, C46, C64, C65, C66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

Commit message: Update RheoBoard v1.05 documentation and manufacturing files. Refined assembly and bringup notes to include updated LED polarity and connector specifications. Corrected footprint and layout details based on recent reviews, ensuring alignment with TI recommendations. Enhanced revision notes to reflect changes in component placements and routing adjustments, including improved via organization and updated BOM references. Manufacturing files, including Gerber and assembly drawings, have been refreshed for accuracy in production.
Parts:
- D13, D14, D15, D17, D19, D6, D7, D8: footprint LED_SMD:LED_0603_1608Metric_Pad1.05x0.95mm_HandSolder -> RheoBoard:LED_SZYY0603R_A1_K2_HandSolder; symbol Device:LED -> RheoBoard_LEDs:SZYY0603R
- D33, D34, D35: footprint LED_SMD:LED_0603_1608Metric -> RheoBoard:LED_SZYY0603R_A1_K2_Nominal; symbol Device:LED -> RheoBoard_LEDs:SZYY0603R
Connections:
- net +4V5: now also D13.1 (A), D14.1 (A); no longer D13.2 (A), D14.2 (A)
- net +6V: now also D17.1 (A), D19.1 (A); no longer D17.2 (A), D19.2 (A)
- net GND: now also D15.2 (K), D33.2 (K), D34.2 (K), D35.2 (K); no longer D15.1 (K), D33.1 (K), D34.1 (K), D35.1 (K)
- net PUMP2_PWM: now also D6.1 (A); no longer D6.2 (A)
- net PUMP3_PWM: now also D7.1 (A); no longer D7.2 (A)
- net PUMP4_PWM: now also D8.1 (A); no longer D8.2 (A)
- net at R40.1: now also D14.2 (K); no longer D14.1 (K)
- net at R54.1: now also D17.2 (K); no longer D17.1 (K)
- net at R24.2: now also D6.2 (K); no longer D6.1 (K)
- net at R59.1: now also D19.2 (K); no longer D19.1 (K)
- net at R44.1: now also D15.1 (A); no longer D15.2 (A)
- net at R77.1: now also D35.1 (A); no longer D35.2 (A)
- net at R73.1: now also D33.1 (A); no longer D33.2 (A)
- net at R25.2: now also D7.2 (K); no longer D7.1 (K)
- net at R39.1: now also D13.2 (K); no longer D13.1 (K)
- net at R26.2: now also D8.2 (K); no longer D8.1 (K)
- net at R75.1: now also D34.1 (A); no longer D34.2 (A)
Changed lines of the file:
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@@
 	)
 	(symbol
-		(lib_id "Device:LED")
+		(lib_id "RheoBoard_LEDs:SZYY0603R")
 		(at 273.05 320.04 0)
 		(unit 1)
@@
 			)
 		)
-		(property "Footprint" "LED_SMD:LED_0603_1608Metric_Pad1.05x0.95mm_HandSolder"
+		(property "Footprint" "RheoBoard:LED_SZYY0603R_A1_K2_HandSolder"
 			(at 273.05 320.04 0)
 			(hide yes)
@@
 			)
 		)
-		(property "Datasheet" ""
+		(property "Datasheet" "https://datasheet.lcsc.com/datasheet/pdf/7948f9a4498910c84f6e992ff3fa9e63.pdf"
 			(at 273.05 320.04 0)
 			(hide yes)
@@
 			)
 		)
-		(property "Description" "Light emitting diode"
+		(property "Description" "SZYY0603R red LED; manufacturer 1=A(+), 2=K(-)"
 			(at 273.05 320.04 0)
 			(hide yes)
@@
 			)
 		)
-		(property "Sim.Pins" "1=K 2=A"
+		(property "Sim.Pins" "1=A 2=K"
 			(at 273.05 320.04 0)
 			(hide yes)
@@
 	)
 	(symbol
-		(lib_id "Device:LED")
+		(lib_id "RheoBoard_LEDs:SZYY0603R")
 		(at 147.32 400.05 0)
 		(unit 1)
@@
 			)
 		)
-		(property "Footprint" "LED_SMD:LED_0603_1608Metric_Pad1.05x0.95mm_HandSolder"
+		(property "Footprint" "RheoBoard:LED_SZYY0603R_A1_K2_HandSolder"
 			(at 147.32 400.05 0)
 			(hide yes)
@@
 			)
 		)
-		(property "Datasheet" ""
+		(property "Datasheet" "https://datasheet.lcsc.com/datasheet/pdf/7948f9a4498910c84f6e992ff3fa9e63.pdf"
 			(at 147.32 400.05 0)
 			(hide yes)
@@
 			)
 		)
-		(property "Description" "Light emitting diode"
+		(property "Description" "SZYY0603R red LED; manufacturer 1=A(+), 2=K(-)"
 			(at 147.32 400.05 0)
 			(hide yes)
@@
 			)
 		)
-		(property "Sim.Pins" "1=K 2=A"
+		(property "Sim.Pins" "1=A 2=K"
 			(at 147.32 400.05 0)
 			(hide yes)
@@
 	)
 	(symbol
-		(lib_id "Device:LED")
+		(lib_id "RheoBoard_LEDs:SZYY0603R")
 		(at 777.24 212.09 180)
 		(unit 1)
@@
 			)
 		)
-		(property "Footprint" "LED_SMD:LED_0603_1608Metric_Pad1.05x0.95mm_HandSolder"
+		(property "Footprint" "RheoBoard:LED_SZYY0603R_A1_K2_HandSolder"
 			(at 777.24 212.09 0)
 			(hide yes)
@@
 			)
 		)
-		(property "Datasheet" ""
+		(property "Datasheet" "https://datasheet.lcsc.com/datasheet/pdf/7948f9a4498910c84f6e992ff3fa9e63.pdf"
 			(at 777.24 212.09 0)
 			(hide yes)
@@
 			)
 		)
-		(property "Description" "Light emitting diode"
+		(property "Description" "SZYY0603R red LED; manufacturer 1=A(+), 2=K(-)"
 			(at 777.24 212.09 0)
 			(hide yes)
@@
 			)
 		)
-		(property "Sim.Pins" "1=K 2=A"
+		(property "Sim.Pins" "1=A 2=K"
 			(at 777.24 212.09 0)
 			(hide yes)
@@
 	)
 	(symbol
-		(lib_id "Device:LED")
+		(lib_id "RheoBoard_LEDs:SZYY0603R")
 		(at 275.59 401.32 0)
 		(unit 1)
@@
 			)
 		)
-		(property "Footprint" "LED_SMD:LED_0603_1608Metric_Pad1.05x0.95mm_HandSolder"
+		(property "Footprint" "RheoBoard:LED_SZYY0603R_A1_K2_HandSolder"
 			(at 275.59 401.32 0)
 			(hide yes)
@@
 			)
 		)
-		(property "Datasheet" ""
+		(property "Datasheet" "https://datasheet.lcsc.com/datasheet/pdf/7948f9a4498910c84f6e992ff3fa9e63.pdf"
 			(at 275.59 401.32 0)
 			(hide yes)
@@
 			)
 		)
-		(property "Description" "Light emitting diode"
+		(property "Description" "SZYY0603R red LED; manufacturer 1=A(+), 2=K(-)"
 			(at 275.59 401.32 0)
 			(hide yes)
@@
 			)
 		)
-		(property "Sim.Pins" "1=K 2=A"
+		(property "Sim.Pins" "1=A 2=K"
 			(at 275.59 401.32 0)
 			(hide yes)
@@
 	)
 	(symbol
-		(lib_id "Device:LED")
+		(lib_id "RheoBoard_LEDs:SZYY0603R")
 		(at 250.19 250.19 90)
 		(unit 1)
@@
 			)
 		)
-		(property "Footprint" "LED_SMD:LED_0603_1608Metric"
+		(property "Footprint" "RheoBoard:LED_SZYY0603R_A1_K2_Nominal"
 			(at 250.19 250.19 0)
 			(hide yes)
@@
 			)
 		)
-		(property "Datasheet" ""
+		(property "Datasheet" "https://datasheet.lcsc.com/datasheet/pdf/7948f9a4498910c84f6e992ff3fa9e63.pdf"
 			(at 250.19 250.19 0)
 			(hide yes)
@@
 			)
 		)
-		(property "Description" "Light emitting diode"
+		(property "Description" "SZYY0603R red LED; manufacturer 1=A(+), 2=K(-)"
 			(at 250.19 250.19 0)
 			(hide yes)
@@
 			)
 		)
-		(property "Sim.Pins" "1=K 2=A"
+		(property "Sim.Pins" "1=A 2=K"
 			(at 250.19 250.19 0)
 			(hide yes)
@@
 	)
 	(symbol
-		(lib_id "Device:LED")
+		(lib_id "RheoBoard_LEDs:SZYY0603R")
 		(at 270.51 95.25 90)
 		(unit 1)
@@
 			)
 		)
-		(property "Footprint" "LED_SMD:LED_0603_1608Metric"
+		(property "Footprint" "RheoBoard:LED_SZYY0603R_A1_K2_Nominal"
 			(at 270.51 95.25 0)
 			(hide yes)
@@
 			)
 		)
-		(property "Datasheet" ""
+		(property "Datasheet" "https://datasheet.lcsc.com/datasheet/pdf/7948f9a4498910c84f6e992ff3fa9e63.pdf"
 			(at 270.51 95.25 0)
 			(hide yes)
@@
 			)
 		)
-		(property "Description" "Light emitting diode"
+		(property "Description" "SZYY0603R red LED; manufacturer 1=A(+), 2=K(-)"
 			(at 270.51 95.25 0)
 			(hide yes)
@@
 			)
 		)
-		(property "Sim.Pins" "1=K 2=A"
+		(property "Sim.Pins" "1=A 2=K"
 			(at 270.51 95.25 0)
 			(hide yes)
@@
 	)
 	(symbol
-		(lib_id "Device:LED")
+		(lib_id "RheoBoard_LEDs:SZYY0603R")
 		(at 777.24 223.52 180)
 		(unit 1)
@@
 			)
 		)
-		(property "Footprint" "LED_SMD:LED_0603_1608Metric_Pad1.05x0.95mm_HandSolder"
+		(property "Footprint" "RheoBoard:LED_SZYY0603R_A1_K2_HandSolder"
 			(at 777.24 223.52 0)
 			(hide yes)
@@
 			)
 		)
-		(property "Datasheet" ""
+		(property "Datasheet" "https://datasheet.lcsc.com/datasheet/pdf/7948f9a4498910c84f6e992ff3fa9e63.pdf"
 			(at 777.24 223.52 0)
 			(hide yes)
@@
 			)
 		)
-		(property "Description" "Light emitting diode"
+		(property "Description" "SZYY0603R red LED; manufacturer 1=A(+), 2=K(-)"
 			(at 777.24 223.52 0)
 			(hide yes)
@@
 			)
 		)
-		(property "Sim.Pins" "1=K 2=A"
+		(property "Sim.Pins" "1=A 2=K"
 			(at 777.24 223.52 0)
 			(hide yes)
@@
 	)
 	(symbol
-		(lib_id "Device:LED")
+		(lib_id "RheoBoard_LEDs:SZYY0603R")
 		(at 146.05 323.85 0)
 		(unit 1)
@@
 			)
 		)
-		(property "Footprint" "LED_SMD:LED_0603_1608Metric_Pad1.05x0.95mm_HandSolder"
+		(property "Footprint" "RheoBoard:LED_SZYY0603R_A1_K2_HandSolder"
 			(at 146.05 323.85 0)
 			(hide yes)
@@
 			)
 		)
-		(property "Datasheet" ""
+		(property "Datasheet" "https://datasheet.lcsc.com/datasheet/pdf/7948f9a4498910c84f6e992ff3fa9e63.pdf"
 			(at 146.05 323.85 0)
 			(hide yes)
@@
 			)
 		)
-		(property "Description" "Light emitting diode"
+		(property "Description" "SZYY0603R red LED; manufacturer 1=A(+), 2=K(-)"
 			(at 146.05 323.85 0)
 			(hide yes)
@@
 			)
 		)
-		(property "Sim.Pins" "1=K 2=A"
+		(property "Sim.Pins" "1=A 2=K"
 			(at 146.05 323.85 0)
 			(hide yes)
@@
 	)
 	(symbol
-		(lib_id "Device:LED")
+		(lib_id "RheoBoard_LEDs:SZYY0603R")
 		(at 817.88 95.25 90)
 		(unit 1)
@@
 			)
 		)
-		(property "Footprint" "LED_SMD:LED_0603_1608Metric_Pad1.05x0.95mm_HandSolder"
+		(property "Footprint" "RheoBoard:LED_SZYY0603R_A1_K2_HandSolder"
 			(at 817.88 95.25 0)
 			(hide yes)
@@
 			)
 		)
-		(property "Datasheet" ""
+		(property "Datasheet" "https://datasheet.lcsc.com/datasheet/pdf/7948f9a4498910c84f6e992ff3fa9e63.pdf"
 			(at 817.88 95.25 0)
 			(hide yes)
@@
 			)
 		)
-		(property "Description" "Light emitting diode"
+		(property "Description" "SZYY0603R red LED; manufacturer 1=A(+), 2=K(-)"
 			(at 817.88 95.25 0)
 			(hide yes)
@@
 			)
 		)
-		(property "Sim.Pins" "1=K 2=A"
+		(property "Sim.Pins" "1=A 2=K"
 			(at 817.88 95.25 0)
 			(hide yes)
@@
 	)
 	(symbol
-		(lib_id "Device:LED")
+		(lib_id "RheoBoard_LEDs:SZYY0603R")
 		(at 777.24 234.95 180)
 		(unit 1)
@@
 			)
 		)
-		(property "Footprint" "LED_SMD:LED_0603_1608Metric_Pad1.05x0.95mm_HandSolder"
+		(property "Footprint" "RheoBoard:LED_SZYY0603R_A1_K2_HandSolder"
 			(at 777.24 234.95 0)
 			(hide yes)
@@
 			)
 		)
-		(property "Datasheet" ""
+		(property "Datasheet" "https://datasheet.lcsc.com/datasheet/pdf/7948f9a4498910c84f6e992ff3fa9e63.pdf"
 			(at 777.24 234.95 0)
 			(hide yes)
@@
 			)
 		)
-		(property "Description" "Light emitting diode"
+		(property "Description" "SZYY0603R red LED; manufacturer 1=A(+), 2=K(-)"
 			(at 777.24 234.95 0)
 			(hide yes)
@@
 			)
 		)
-		(property "Sim.Pins" "1=K 2=A"
+		(property "Sim.Pins" "1=A 2=K"
 			(at 777.24 234.95 0)
 			(hide yes)
@@
 	)
 	(symbol
-		(lib_id "Device:LED")
+		(lib_id "RheoBoard_LEDs:SZYY0603R")
 		(at 247.65 171.45 90)
 		(unit 1)
@@
 			)
 		)
-		(property "Footprint" "LED_SMD:LED_0603_1608Metric"
+		(property "Footprint" "RheoBoard:LED_SZYY0603R_A1_K2_Nominal"
 			(at 247.65 171.45 0)
 			(hide yes)
@@
 			)
 		)
-		(property "Datasheet" ""
+		(property "Datasheet" "https://datasheet.lcsc.com/datasheet/pdf/7948f9a4498910c84f6e992ff3fa9e63.pdf"
 			(at 247.65 171.45 0)
 			(hide yes)
@@
 			)
 		)
-		(property "Description" "Light emitting diode"
+		(property "Description" "SZYY0603R red LED; manufacturer 1=A(+), 2=K(-)"
 			(at 247.65 171.45 0)
 			(hide yes)
@@
 			)
 		)
-		(property "Sim.Pins" "1=K 2=A"
+		(property "Sim.Pins" "1=A 2=K"
 			(at 247.65 171.45 0)
 			(hide yes)

Commit message: Update RheoBoard v1.05 documentation and remove obsolete files. Enhanced README for clarity on project versions and updated assembly notes. Removed outdated files related to v0.05-altium and v1.05, including assembly and footprint documentation, to streamline project structure. Added local ignore rules for PCB diagnostics and updated BOM references for accuracy in production.
Parts:
- J3: footprint Connector_JST:JST_EH_B4B-EH-A_1x04_P2.50mm_Vertical -> RheoBoard:JST_EH_B4B-EH-A_1x04_P2.50mm_Vertical_DFM
- Q11: footprint Package_TO_SOT_SMD:SOT-223-3_TabPin2 -> RheoBoard:SOT-223-3_TabPin2_DFM
- Q3: footprint RheoBoard:AO3400A -> RheoBoard:AO3400A_Pin1Offset
Changed lines of the file:
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@@
 			)
 		)
-		(property "Footprint" "Package_TO_SOT_SMD:SOT-223-3_TabPin2"
+		(property "Footprint" "RheoBoard:SOT-223-3_TabPin2_DFM"
 			(at 95.25 68.58 0)
 			(hide yes)
@@
 			)
 		)
-		(property "Footprint" "Connector_JST:JST_EH_B4B-EH-A_1x04_P2.50mm_Vertical"
+		(property "Footprint" "RheoBoard:JST_EH_B4B-EH-A_1x04_P2.50mm_Vertical_DFM"
 			(at 840.74 163.83 0)
 			(hide yes)
@@
 			)
 		)
-		(property "Footprint" "RheoBoard:AO3400A"
+		(property "Footprint" "RheoBoard:AO3400A_Pin1Offset"
 			(at 110.49 354.33 0)
 			(hide yes)

Commit message: Update RheoBoard v1.05 manufacturing files and documentation. Refreshed BOM, Gerber, and assembly drawings with updated creation timestamps. Enhanced component descriptions and assembly notes for clarity and accuracy. Adjusted designators and added new properties for improved organization and documentation consistency.
Parts:
- D36: Assembly Notes (none) -> Exact Littelfuse SMBJ13A (not SMBJ13CA or SMBJ14A); marking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; VBR (none) -> 14.4-15.9 V at 1 mA; VC (none) -> 21.5 V max at 28 A (10/1000 us); VRWM (none) -> 13 V
- J19: Assembly Notes (none) -> Fit one 5-position segment cut from Adafruit 392 36-pin str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; MPN 1x05_2.54mm_vertical_header -> 392; Manufacturer Generic -> Adafruit Industries LLC; Source (none) -> https://www.adafruit.com/product/392
Changed lines of the file:
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@@
 			)
 		)
-		(property "Datasheet" ""
+		(property "Datasheet" "https://www.adafruit.com/product/392"
 			(at 586.74 93.98 0)
 			(hide yes)
@@
 			)
 		)
-		(property "Description" "5-pin button GPIO header; GND, SW1, SW2, SW3, SW4. Pull-ups powered by HOST_3V3 via J9."
+		(property "Description" "Adafruit 392 straight 2.54 mm breakaway male header, cut to 5 positions. Pins 1-5: GND, VALVE1_IN, VALVE2_IN, PUMP1_IN, PUMP2_IN. Pullups use HOST_3V3 via J9; no power pin."
 			(at 586.74 93.98 0)
 			(hide yes)
@@
 			)
 		)
-		(property "MPN" "1x05_2.54mm_vertical_header"
+		(property "MPN" "392"
 			(at 586.74 93.98 0)
 			(hide yes)
@@
 			)
 		)
-		(property "Manufacturer" "Generic"
+		(property "Manufacturer" "Adafruit Industries LLC"
 			(at 586.74 93.98 0)
 			(hide yes)
@@
 			)
 		)
-		(property "Source" ""
+		(property "Source" "https://www.adafruit.com/product/392"
 			(at 586.74 93.98 0)
 			(hide yes)
@@
 			)
 		)
-	)
+		(property "Assembly Notes" "Fit one 5-position segment cut from Adafruit 392 36-pin strip (10 strips per retail pack). Pin 1 is square/GND. Manual through-hole assembly; check cut-end integrity and mating cable fit."
+			(at 586.74 93.98 0)
+			(hide yes)
+			(effects
+				(font
+					(size 1.27 1.27)
+				)
+			)
+		))
 	(symbol
 		(lib_id "Mechanical:MountingHole")
@@
 			)
 		)
-		(property "Datasheet" "https://m.littelfuse.com/~/media/electronics/datasheets/tvs_diodes/littelfuse_tvs_diode_smbj_datasheet.pdf.pdf"
+		(property "Datasheet" "https://www.littelfuse.com/assetdocs/tvs-diodes-smbj-series-datasheet?assetguid=ba555e99-a12d-4f72-a0b6-86b06c67171e"
 			(at 408.94 90.17 0)
 			(hide yes)
@@
 			)
 		)
-		(property "Description" "Zener diode"
+		(property "Description" "Unidirectional TVS, Littelfuse SMBJ13A, 13 V standoff, 600 W (10/1000 us), DO-214AA (SMB); cathode pad 1 to VIN_RAW, anode pad 2 to GND."
 			(at 408.94 90.17 0)
 			(hide yes)
@@
 			)
 		)
-	)
+		(property "Assembly Notes" "Exact Littelfuse SMBJ13A (not SMBJ13CA or SMBJ14A); marking LG; cathode band at pad 1 / VIN_RAW. Manufacturer ratings override conflicting distributor headline."
+			(at 408.94 90.17 0)
+			(hide yes)
+			(effects
+				(font
+					(size 1.27 1.27)
+				)
+			)
+		)
+		(property "VBR" "14.4-15.9 V at 1 mA"
+			(at 408.94 90.17 0)
+			(hide yes)
+			(effects
+				(font
+					(size 1.27 1.27)
+				)
+			)
+		)
+		(property "VC" "21.5 V max at 28 A (10/1000 us)"
+			(at 408.94 90.17 0)
+			(hide yes)
+			(effects
+				(font
+					(size 1.27 1.27)
+				)
+			)
+		)
+		(property "VRWM" "13 V"
+			(at 408.94 90.17 0)
+			(hide yes)
+			(effects
+				(font
+					(size 1.27 1.27)
+				)
+			)
+		))
 	(symbol
 		(lib_id "RheoBoard_LEDs:SZYY0603R")
