File: RheoBoard_PCB/RheoBoard_v1.05/RheoBoard_v1.05/RheoBoard_v1.05.kicad_sch (KiCad schematic)
At the start: 160 parts, among them J1 JST SH 4-pin 1.00mm, J12 JST SH 4-pin 1.00mm, J17 JST SH 4-pin 1.00mm, J19 BUTTONS_GPIO, J2 PJ-082BH, J3 JST EH 4-pin 2.50mm, J9 JST SH 4-pin 1.00mm, Q10 AO3400A, Q11 DMP6023LE-13, Q3 AO3400A, Q4 AO3400A, Q8 AO3400A, SW1 TL3301NF160QG/P010515, SW2 TL3301NF160QG/P010515, SW3 TL3301NF160QG/P010515, SW4 TL3301NF160QG/P010515, U1 TPS563203DRLR, U10 JST XH 2-pin 2.50mm, U11 ZR370-02PM / 4.5V / 2.5 LPM /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, U12 TPS259472ARPWR, U13 TCA9517ADGKR, U2 TPS563203DRLR, U3 TPS563203DRLR, U5 MPRLS0025PA00001A, U7 PCA9685PW,118, U8 ZR370-02PM / 4.5V / 2.5 LPM /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, U9 JST XH 2-pin 2.50mm

Commit message: Update BOM and schematic properties for RheoBoard v1.05. Adjusted component values, LCSC part numbers, and descriptions for capacitors and resistors. Enhanced clarity and accuracy in documentation, including updated creation timestamps for manufacturing files.
Parts:
- C55, C58: value 18pF 50V C0G ±2% -> 18pF 50V C0G ±5%; LCSC C2169079 -> C107040; MPN VJ0603A180GXACW1BC -> CC0603JRNPO9BN180; Manufacturer VISHAY -> YAGEO; Source https://www.lcsc.com/product-detail/C2169079.html -> https://www.lcsc.com/product-detail/C107040.html
- C62: value 18pF 50V C0G ±2% -> 24pF 50V C0G ±5%; LCSC C2169079 -> C107044; MPN VJ0603A180GXACW1BC -> CC0603JRNPO9BN240; Manufacturer VISHAY -> YAGEO; Source https://www.lcsc.com/product-detail/C2169079.html -> https://www.lcsc.com/product-detail/C107044.html
- J19: Assembly Notes Fit one 5-position segment cut from Adafruit 392 36-pin str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 -> Fit complete five-pin header C124379. Pin 1 is square/GND. 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; LCSC (none) -> C124379; MPN 392 -> B-2100S05P-A110; Manufacturer Adafruit Industries LLC -> Ckmtw; Source https://www.adafruit.com/product/392 -> https://www.lcsc.com/product-detail/C124379.html
- R61: value 135k ±0.1% -> 100k ±1%; LCSC C861113 -> C25803; MPN RT0603BRD07135KL -> 0603WAF1003T5E; Manufacturer YAGEO -> UNI-ROYAL; Source https://www.lcsc.com/product-detail/C861113.html -> https://www.lcsc.com/product-detail/C25803.html
- R73: value 549R ±1% -> 560R ±1%; LCSC C23079 -> C23204; MPN 0603WAF5490T5E -> 0603WAF5600T5E; Source https://www.lcsc.com/product-detail/C23079.html -> https://www.lcsc.com/product-detail/C23204.html
- R76: value 30K/0603/1% -> 22k ±1%; LCSC C22984 -> C31850; MPN 0603WAF3002T5E -> 0603WAF2202T5E; Source https://www.lcsc.com/product-detail/C22984.html -> https://www.lcsc.com/product-detail/C31850.html
Changed lines of the file:
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@@
 			)
 		)
-		(property "Value" "135k ±0.1%"
+		(property "Value" "100k ±1%"
 			(at 214.122 236.474 90)
 			(show_name no)
@@
 			)
 		)
-		(property "LCSC" "C861113"
+		(property "LCSC" "C25803"
 			(at 209.55 236.22 0)
 			(hide yes)
@@
 			)
 		)
-		(property "MPN" "RT0603BRD07135KL"
+		(property "MPN" "0603WAF1003T5E"
 			(at 209.55 236.22 0)
 			(hide yes)
@@
 			)
 		)
-		(property "Manufacturer" "YAGEO"
+		(property "Manufacturer" "UNI-ROYAL"
 			(at 209.55 236.22 0)
 			(hide yes)
@@
 			)
 		)
-		(property "Source" "https://www.lcsc.com/product-detail/C861113.html"
+		(property "Source" "https://www.lcsc.com/product-detail/C25803.html"
 			(at 209.55 236.22 0)
 			(hide yes)
@@
 			)
 		)
-		(property "Datasheet" "https://www.adafruit.com/product/392"
+		(property "Datasheet" "https://datasheet.lcsc.com/datasheet/pdf/219f7e7eb5f34457895b2c164313179f.pdf?productCode=C124379"
 			(at 586.74 93.98 0)
 			(hide yes)
@@
 			)
 		)
-		(property "Description" "Adafruit 392 straight 2.54 mm breakaway male header, cut to 5 positions. Pins 1-5: GND, VALVE1_IN, VALVE2_IN, PUMP1_IN, PUMP2_IN. Pullups use HOST_3V3 via J9; no power pin."
+		(property "Description" "Ckmtw B-2100S05P-A110 straight 1x05 2.54 mm male header. Pins 1-5: GND, VALVE1_IN, VALVE2_IN, PUMP1_IN, PUMP2_IN. Pullups use HOST_3V3 via J9; no power pin."
 			(at 586.74 93.98 0)
 			(hide yes)
@@
 			)
 		)
-		(property "LCSC" ""
+		(property "LCSC" "C124379"
 			(at 586.74 93.98 0)
 			(hide yes)
@@
 			)
 		)
-		(property "MPN" "392"
+		(property "MPN" "B-2100S05P-A110"
 			(at 586.74 93.98 0)
 			(hide yes)
@@
 			)
 		)
-		(property "Manufacturer" "Adafruit Industries LLC"
+		(property "Manufacturer" "Ckmtw"
 			(at 586.74 93.98 0)
 			(hide yes)
@@
 			)
 		)
-		(property "Source" "https://www.adafruit.com/product/392"
+		(property "Source" "https://www.lcsc.com/product-detail/C124379.html"
 			(at 586.74 93.98 0)
 			(hide yes)
@@
 			)
 		)
-		(property "Assembly Notes" "Fit one 5-position segment cut from Adafruit 392 36-pin strip (10 strips per retail pack). Pin 1 is square/GND. Manual through-hole assembly; check cut-end integrity and mating cable fit."
+		(property "Assembly Notes" "Fit complete five-pin header C124379. Pin 1 is square/GND. Manual through-hole assembly; 0.60 mm square pins, 3 mm tails, 6 mm mating pins. Existing footprint retained."
 			(at 586.74 93.98 0)
 			(hide yes)
@@
 			)
 		)
-		(property "Value" "18pF 50V C0G ±2%"
+		(property "Value" "18pF 50V C0G ±5%"
 			(at 223.266 165.1 90)
 			(show_name no)
@@
 			)
 		)
-		(property "LCSC" "C2169079"
+		(property "LCSC" "C107040"
 			(at 218.44 154.94 0)
 			(hide yes)
@@
 			)
 		)
-		(property "MPN" "VJ0603A180GXACW1BC"
+		(property "MPN" "CC0603JRNPO9BN180"
 			(at 218.44 154.94 0)
 			(hide yes)
@@
 			)
 		)
-		(property "Manufacturer" "VISHAY"
+		(property "Manufacturer" "YAGEO"
 			(at 218.44 154.94 0)
 			(hide yes)
@@
 			)
 		)
-		(property "Source" "https://www.lcsc.com/product-detail/C2169079.html"
+		(property "Source" "https://www.lcsc.com/product-detail/C107040.html"
 			(at 218.44 154.94 0)
 			(hide yes)
@@
 			)
 		)
-		(property "Value" "18pF 50V C0G ±2%"
+		(property "Value" "24pF 50V C0G ±5%"
 			(at 227.076 246.38 90)
 			(show_name no)
@@
 			)
 		)
-		(property "LCSC" "C2169079"
+		(property "LCSC" "C107044"
 			(at 222.25 236.22 0)
 			(hide yes)
@@
 			)
 		)
-		(property "MPN" "VJ0603A180GXACW1BC"
+		(property "MPN" "CC0603JRNPO9BN240"
 			(at 222.25 236.22 0)
 			(hide yes)
@@
 			)
 		)
-		(property "Manufacturer" "VISHAY"
+		(property "Manufacturer" "YAGEO"
 			(at 222.25 236.22 0)
 			(hide yes)
@@
 			)
 		)
-		(property "Source" "https://www.lcsc.com/product-detail/C2169079.html"
+		(property "Source" "https://www.lcsc.com/product-detail/C107044.html"
 			(at 222.25 236.22 0)
 			(hide yes)
@@
 			)
 		)
-		(property "Value" "18pF 50V C0G ±2%"
+		(property "Value" "18pF 50V C0G ±5%"
 			(at 249.428 94.488 90)
 			(show_name no)
@@
 			)
 		)
-		(property "LCSC" "C2169079"
+		(property "LCSC" "C107040"
 			(at 243.84 81.28 0)
 			(hide yes)
@@
 			)
 		)
-		(property "MPN" "VJ0603A180GXACW1BC"
+		(property "MPN" "CC0603JRNPO9BN180"
 			(at 243.84 81.28 0)
 			(hide yes)
@@
 			)
 		)
-		(property "Manufacturer" "VISHAY"
+		(property "Manufacturer" "YAGEO"
 			(at 243.84 81.28 0)
 			(hide yes)
@@
 			)
 		)
-		(property "Source" "https://www.lcsc.com/product-detail/C2169079.html"
+		(property "Source" "https://www.lcsc.com/product-detail/C107040.html"
 			(at 243.84 81.28 0)
 			(hide yes)
@@
 			)
 		)
-		(property "Value" "30K/0603/1%"
+		(property "Value" "22k ±1%"
 			(at 220.726 255.27 0)
 			(show_name no)
@@
 			)
 		)
-		(property "LCSC" "C22984"
+		(property "LCSC" "C31850"
 			(at 209.55 255.27 0)
 			(hide yes)
@@
 			)
 		)
-		(property "MPN" "0603WAF3002T5E"
+		(property "MPN" "0603WAF2202T5E"
 			(at 209.55 255.27 0)
 			(hide yes)
@@
 			)
 		)
-		(property "Source" "https://www.lcsc.com/product-detail/C22984.html"
+		(property "Source" "https://www.lcsc.com/product-detail/C31850.html"
 			(at 209.55 255.27 0)
 			(hide yes)
@@
 			)
 		)
-		(property "Value" "549R ±1%"
+		(property "Value" "560R ±1%"
 			(at 273.812 79.248 90)
 			(show_name no)
@@
 			)
 		)
-		(property "LCSC" "C23079"
+		(property "LCSC" "C23204"
 			(at 270.51 80.01 0)
 			(hide yes)
@@
 			)
 		)
-		(property "MPN" "0603WAF5490T5E"
+		(property "MPN" "0603WAF5600T5E"
 			(at 270.51 80.01 0)
 			(hide yes)
@@
 			)
 		)
-		(property "Source" "https://www.lcsc.com/product-detail/C23079.html"
+		(property "Source" "https://www.lcsc.com/product-detail/C23204.html"
 			(at 270.51 80.01 0)
 			(hide yes)

Commit message: Update BOM and manufacturing files for RheoBoard v1.05. Adjusted component values, added new components, and corrected designator placements. Updated creation timestamps for Gerber and manufacturing files to reflect the latest changes.
Parts:
- added C70: 100nF 50V X7R ±10%, Capacitor_SMD:C_0603_1608Metric, symbol Device:C
- added U14: TLV803EA29DBZR, Package_TO_SOT_SMD:SOT-23, symbol RheoBoard_Fixes:TLV803EA29DBZR
- C58: value 18pF 50V C0G ±5% -> 20pF 50V C0G ±5%; LCSC C107040 -> C1648; MPN CC0603JRNPO9BN180 -> CL10C200JB8NNNC; Manufacturer YAGEO -> Samsung Electro-Mechanics; Source https://www.lcsc.com/product-detail/C107040.html -> https://www.lcsc.com/product-detail/C1648.html
- R60: value 270K/0603/1% -> 240k ±1%; LCSC C22965 -> C4197; MPN 0603WAF2703T5E -> 0603WAF2403T5E; Source https://www.lcsc.com/product-detail/C22965.html -> https://www.lcsc.com/product-detail/C4197.html
Connections:
- net +3V3: now also C70.1, U14.3 (VDD)
- net GND: now also C70.2, U14.1 (GND)
- net RES: now also U14.2 (~{RESET})
- net +6V renamed +5V4
Other:
- note added: "BUCK 12V - 5V4"
- note removed: "BUCK 12V - 6V"
