File: RheoBoard_PCB/RheoBoard_v1.05/RheoBoard_v1.05/RheoBoard_v1.05.kicad_pcb (KiCad board)
At the start: 2 copper layers, 109 x 126.4 mm, 160 parts, among them J1 JST SH 4-pin 1.00mm, J12 JST SH 4-pin 1.00mm, J17 JST SH 4-pin 1.00mm, J19 BUTTONS_GPIO, J2 PJ-082BH, J3 JST EH 4-pin 2.50mm, J9 JST SH 4-pin 1.00mm, Q10 AO3400A, Q11 DMP6023LE-13, Q3 AO3400A, Q4 AO3400A, Q8 AO3400A, SW1 TL3301NF160QG/P010515, SW2 TL3301NF160QG/P010515, SW3 TL3301NF160QG/P010515, SW4 TL3301NF160QG/P010515, U1 TPS563203DRLR, U10 JST XH 2-pin 2.50mm, U11 ZR370-02PM / 4.5V / 2.5 LPM /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, U12 TPS259472ARPWR, U13 TCA9517ADGKR, U2 TPS563203DRLR, U3 TPS563203DRLR, U5 MPRLS0025PA00001A, U7 PCA9685PW,118, U8 ZR370-02PM / 4.5V / 2.5 LPM /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, U9 JST XH 2-pin 2.50mm

Commit message: Improve v1.05 power routing and refresh manufacturing files
Routing:
- net GND: vias 263 -> 275
