File: RheoBoard_PCB/RheoBoard_v1.05/RheoBoard_v1.05/RheoBoard_v1.05.kicad_pcb (KiCad board)
At the start: 2 copper layers, 109 x 126.4 mm, 160 parts, among them J1 JST SH 4-pin 1.00mm, J12 JST SH 4-pin 1.00mm, J17 JST SH 4-pin 1.00mm, J19 BUTTONS_GPIO, J2 PJ-082BH, J3 JST EH 4-pin 2.50mm, J9 JST SH 4-pin 1.00mm, Q10 AO3400A, Q11 DMP6023LE-13, Q3 AO3400A, Q4 AO3400A, Q8 AO3400A, SW1 TL3301NF160QG/P010515, SW2 TL3301NF160QG/P010515, SW3 TL3301NF160QG/P010515, SW4 TL3301NF160QG/P010515, U1 TPS563203DRLR, U10 JST XH 2-pin 2.50mm, U11 ZR370-02PM / 4.5V / 2.5 LPM /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, U12 TPS259472ARPWR, U13 TCA9517ADGKR, U2 TPS563203DRLR, U3 TPS563203DRLR, U5 MPRLS0025PA00001A, U7 PCA9685PW,118, U8 ZR370-02PM / 4.5V / 2.5 LPM /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, U9 JST XH 2-pin 2.50mm

Commit message: Improve v1.05 silkscreen labels and refresh manufacturing files
Other:
- board text added: "3V3"
- board text added: "C1"
- board text added: "C15"
- board text added: "C23"
- board text added: "C24"
- board text added: "C25"
- board text added: "C26"
- board text added: "C27"
- board text added: "C28"
- board text added: "C29"
- board text added: "C31"
- board text added: "C32"
- board text added: "C33"
- board text added: "C34"
- board text added: "C43"
- board text added: "C45"
- board text added: "C46"
- board text added: "C53"
- board text added: "C55"
- board text added: "C56"
- board text added: "C58"
- board text added: "C59"
- board text added: "C61"
- board text added: "C62"
- board text added: "C63"
- board text added: "C65"
- board text added: "C66"
- board text added: "C67"
- board text added: "C8"
- board text added: "D11"
- board text added: "D12"
- board text added: "D15"
- board text added: "D16"
- board text added: "D18"
- board text added: "D34"
- board text added: "D35"
- board text added: "D36"
- board text added: "D6"
- board text added: "D7"
- board text added: "D8"
- board text added: "J1"
- board text added: "J12"
- board text added: "J17"
- board text added: "J2"
- board text added: "J3"
- board text added: "JP2"
- board text added: "JP3"
- board text added: "JP4"
- board text added: "JP5"
- board text added: "JP6"
- board text added: "JP7"
- board text added: "L1"
- board text added: "L2"
- board text added: "L5"
- board text added: "PUMP U11"
- board text added: "PUMP U8"
- board text added: "Q10"
- board text added: "Q8"
- board text added: "R1"
- board text added: "R15"
- board text added: "R20"
- board text added: "R22"
- board text added: "R23"
- board text added: "R24"
- board text added: "R25"
- board text added: "R29"
- board text added: "R30"
- board text added: "R31"
- board text added: "R32"
- board text added: "R33"
- board text added: "R34"
- board text added: "R35"
- board text added: "R36"
- board text added: "R38"
- board text added: "R4"
- board text added: "R54"
- board text added: "R55"
- board text added: "R59"
- board text added: "R7"
- board text added: "R73"
- board text added: "R75"
- board text added: "R77"
- board text added: "R80"
- board text added: "SW1"
- board text added: "SW2"
- board text added: "SW3"
- board text added: "SW4"
- board text added: "TP2"
- board text added: "TP4"
- board text added: "TP5"
- board text added: "TP6"
- board text added: "TP7"
- board text added: "TP8"
- board text added: "TP9"
- board text added: "U5"
- board text added: "U7"
- board text added: "VALVE U10"
- board text added: "VALVE U9"
- board text removed: "+3V3"
- board text removed: "3V3 OUT"
- board text removed: "HOST 3V3 IN"

Commit message: Update BOM and schematic properties for RheoBoard v1.05. Adjusted component values, LCSC part numbers, and descriptions for capacitors and resistors. Enhanced clarity and accuracy in documentation, including updated creation timestamps for manufacturing files.
Parts:
- C55, C58: value 18pF 50V C0G ±2% -> 18pF 50V C0G ±5%
- C62: value 18pF 50V C0G ±2% -> 24pF 50V C0G ±5%
- R61: value 135k ±0.1% -> 100k ±1%
- R73: value 549R ±1% -> 560R ±1%
- R76: value 30K/0603/1% -> 22k ±1%

Commit message: Update BOM and manufacturing files for RheoBoard v1.05. Adjusted component values, added new components, and corrected designator placements. Updated creation timestamps for Gerber and manufacturing files to reflect the latest changes.
Parts:
- added C70: 100nF 50V X7R ±10%, Capacitor_SMD:C_0603_1608Metric, F.Cu at (139.0, 81.5)
- added U14: TLV803EA29DBZR, Package_TO_SOT_SMD:SOT-23, F.Cu at (137.5, 85.0)
- C58: value 18pF 50V C0G ±5% -> 20pF 50V C0G ±5%
- R60: value 270K/0603/1% -> 240k ±1%
Connections:
- net +6V renamed +5V4
Routing:
- net /RES: track 3.55 -> 16.9 mm, vias 0 -> 1
- net +3V3: track 323.4 -> 333.7 mm
- net GND: track 7.76 -> 9.78 mm, vias 275 -> 277
Other:
- board text added: "QWIIC HOST"
- board text added: "QWIIC SENSOR"
